Commit message: visual processing updated

File: flexbotics_cr7ial_support/urdf/cr7ial_scene.urdf.xacro (robot description, xacro)
@@ -46,6 +46,7 @@
   <!-- Camera -->
   <xacro:include filename="$(find realsense2_description)/urdf/_d435.urdf.xacro" />
-  <xacro:sensor_d435 name="camera" parent="sensors_assembly">
-	  <origin xyz="0 0.139 0.13" rpy="3.14 -0.031 1.582" />
+  <xacro:sensor_d435 name="camera" parent="tool0" use_nominal_extrinsics="true">
+	  <origin xyz="0.13 -0.045 0.13" rpy="3.14 -0.031 -0.34" />
+    <!-- <origin xyz="0.06 -0.05 0.041" rpy="-0.061 -0.068 1.564" /> -->
 	</xacro:sensor_d435>
 </robot>

Commit message: gazebo updated without gravity

File: flexbotics_cr7ial_support/urdf/cr7ial_scene.urdf.xacro (robot description, xacro)
@@ -1,9 +1,9 @@
-<?xml version="1.0" ?>
-<robot name="calibration_scene" xmlns:xacro="http://ros.org/wiki/xacro">
+<?xml version="1.0"?>
+<robot xmlns:xacro="http://wiki.ros.org/xacro" name="calibration_scene">
   <!--world -->
   <link name="world"/>
-  <!-- Import robot -->
-  <xacro:include filename="$(find fanuc_cr7ia_support)/urdf/cr7ial_macro.xacro"/>
-  <xacro:fanuc_cr7ial prefix=""/>
+  <!-- Import robot model macro and instantiate -->
+  <xacro:include filename="$(find fanuc_cr7ial_gazebo_support)/urdf/fanuc_cr7ial_gazebo.xacro" />
+  <xacro:fanuc_cr7ial prefix="" />
   <!-- Import end effector -->
   <xacro:include filename="$(find flexbotics_cr7ial_support)/urdf/cr7ial_scan_blend_eff_macro.xacro"/>
@@ -33,6 +33,6 @@
   </joint>
   <!-- Place robot on top of the table -->
-  <joint name="base_to_table" type="fixed">
-    <parent link="table"/>
+  <joint name="world " type="fixed">
+    <parent link="world"/>
     <child link="base_link"/>
     <origin xyz="0.4 0.0 0.8" rpy="0.0 0.0 0.0"/>
@@ -46,7 +46,11 @@
   <!-- Camera -->
   <xacro:include filename="$(find realsense2_description)/urdf/_d435.urdf.xacro" />
-  <xacro:sensor_d435 name="camera" parent="tool0" use_nominal_extrinsics="true">
+  <xacro:sensor_d435 name="camera" parent="tool0" >
 	  <origin xyz="0.13 -0.045 0.13" rpy="3.14 -0.031 -0.34" />
-    <!-- <origin xyz="0.06 -0.05 0.041" rpy="-0.061 -0.068 1.564" /> -->
 	</xacro:sensor_d435>
+  <gazebo reference="camera_link">
+    <turnGravityOff>true</turnGravityOff>
+  </gazebo>
+  <!-- Add Gazebo ROS-control (include only once in your project) -->
+  <xacro:include filename="$(find fanuc_gazebo_common)/urdf/fanuc_ros_control_gazebo.xacro" />
 </robot>

Commit message: moveit move_group implemented

File: flexbotics_cr7ial_support/urdf/cr7ial_scene.urdf.xacro (robot description, xacro)
@@ -12,5 +12,5 @@
   <link name="table">
     <visual>
-      <origin xyz="1.0 0.0 0.4"/>
+      <origin xyz="0.5 0.0 0.4"/>
       <geometry>
         <box size="2.0 1.0 0.8"/>
@@ -21,5 +21,5 @@
     </visual>
     <collision>
-      <origin xyz="1.0 0.0 0.4"/>
+      <origin xyz="0.5 0.0 0.4"/>
       <geometry>
         <box size="2.0 1.0 0.8"/>
@@ -36,5 +36,5 @@
     <parent link="world"/>
     <child link="base_link"/>
-    <origin xyz="0.4 0.0 0.8" rpy="0.0 0.0 0.0"/>
+    <origin xyz="0 0.0 0.8" rpy="0.0 0.0 0.0"/>
   </joint>
   <!-- Place sensors end effector on robot flange -->

Commit message: remove end effector

File: flexbotics_cr7ial_support/urdf/cr7ial_scene.urdf.xacro (robot description, xacro)
@@ -7,6 +7,6 @@
   <xacro:fanuc_cr7ial prefix="" />
   <!-- Import end effector -->
-  <xacro:include filename="$(find flexbotics_cr7ial_support)/urdf/cr7ial_scan_blend_eff_macro.xacro"/>
-  <xacro:sensors_end_effector prefix=""/>
+  <!-- <xacro:include filename="$(find flexbotics_cr7ial_support)/urdf/cr7ial_scan_blend_eff_macro.xacro"/>
+  <xacro:sensors_end_effector prefix=""/> -->
   <!-- Table where the robot and calibration plane will be placed -->
   <link name="table">
@@ -39,9 +39,9 @@
   </joint>
   <!-- Place sensors end effector on robot flange -->
-  <joint name="robot_tool0_to_sensors_eff" type="fixed">
+  <!-- <joint name="robot_tool0_to_sensors_eff" type="fixed">
     <parent link="tool0"/>
     <child link="eff_frame"/>
     <origin xyz="0 0 0" rpy="0 0 0"/>
-  </joint>
+  </joint> -->
   <!-- Camera -->
   <xacro:include filename="$(find realsense2_description)/urdf/_d435.urdf.xacro" />

Commit message: transformation matrix updated

File: flexbotics_cr7ial_support/urdf/cr7ial_scene.urdf.xacro (robot description, xacro)
@@ -9,4 +9,7 @@
   <!-- <xacro:include filename="$(find flexbotics_cr7ial_support)/urdf/cr7ial_scan_blend_eff_macro.xacro"/>
   <xacro:sensors_end_effector prefix=""/> -->
+  <!-- Import end effector -->
+  <!-- <xacro:include filename="$(find flexbotics_cr7ial_support)/urdf/PhoXi3Dscanner.xacro"/>
+  <xacro:PhoXi3Dscanner prefix=""/> -->
   <!-- Table where the robot and calibration plane will be placed -->
   <link name="table">
@@ -47,5 +50,5 @@
   <xacro:include filename="$(find realsense2_description)/urdf/_d435.urdf.xacro" />
   <xacro:sensor_d435 name="camera" parent="tool0" >
-	  <origin xyz="0.13 -0.045 0.13" rpy="3.14 -0.031 -0.34" />
+	  <origin xyz=" 0.02268366 -0.0958564   0.07088306" rpy=" 1.59691407 -1.56299734  0.39588142" />
 	</xacro:sensor_d435>
   <gazebo reference="camera_link">
